Commit message: add geometry_msgs::Twist control: rostopic "/nubot_drive/base_auto_cmd"

File: gazebo_description/models/NuBot_Pumbaa_v2/model_v2.urdf.xacro (robot description, xacro)
@@ -23,5 +23,5 @@
                  izz="0.319921" />
       </inertial>
-      <collision name='base_link_collision_1'>
+      <collision name='base_collision_1'>
         <origin xyz="${track_length/2} 0 0" rpy="${PI/2} 0 0" />
         <geometry>
@@ -29,5 +29,5 @@
         </geometry>
       </collision>
-      <collision name='base_link_collision_2'>
+      <collision name='base_collision_2'>
         <origin xyz="${-1*track_length/2} 0 0" rpy="${PI/2} 0 0" />
         <geometry>
@@ -35,5 +35,5 @@
         </geometry>
       </collision>
-      <collision name='base_link_collision'>
+      <collision name='base_collision'>
         <origin xyz="0 0 0" rpy="0 0 0" />
         <geometry>
@@ -41,5 +41,5 @@
         </geometry>
       </collision>
-      <visual name='base_link_visual'>
+      <visual name='base_visual'>
         <origin xyz="0 0 0" rpy="0 0 0" />
         <geometry>
@@ -47,5 +47,5 @@
         </geometry>
       </visual>
-      <visual name='base_link_vive_link_visual'>
+      <visual name='base_vive_link_visual'>
         <origin xyz="0.16175 0 0.138" rpy="0 0 0" />
         <geometry>
@@ -55,12 +55,14 @@
     </link>
     <gazebo reference="base_link">
-      <self_collide>false</self_collide>
+      <selfCollide>false</selfCollide>
       <mu1>1</mu1>
       <mu2>1</mu2>
       <fdir1 value="0 1 0" />
       <gravity>1</gravity>
-      <kinematic>0</kinematic>
-      <enable_wind>0</enable_wind>
-      <max_contacts>10</max_contacts>
+      <maxContacts>10</maxContacts>
+      <plugin name='NuBot_Pumbaa_Gazebo_Plugin' filename='libnubot_pumbaa_plugin.so'>
+        <!--The link tags of tracks-->
+        <!-- <body>base_link</body> -->
+      </plugin>
     </gazebo>
     <!--left_track-->
@@ -99,12 +101,14 @@
       </collision>
       <gazebo reference="left_track_link">
-        <self_collide>false</self_collide>
-        <mu1>0.7</mu1>
-        <mu2>150</mu2>
-        <fdir1 value="0 1 0" />
-        <gravity>1</gravity>
-        <kinematic>0</kinematic>
-        <enable_wind>0</enable_wind>
-        <max_contacts>10</max_contacts>
+        <selfCollide>false</selfCollide>
+        <mu1>0.7</mu1>
+        <mu2>150</mu2>
+        <fdir1 value="0 1 0" />
+        <gravity>1</gravity>
+        <maxContacts>10</maxContacts>
+        <plugin name='NuBot_Pumbaa_Gazebo_Plugin' filename='libnubot_pumbaa_plugin.so'>
+          <!--The link tags of tracks-->
+          <!-- <left_track>left_track_link</left_track> -->
+        </plugin>
       </gazebo>
     </link>
@@ -144,12 +148,14 @@
       </collision>
       <gazebo reference="right_track_link">
-        <self_collide>false</self_collide>
-        <mu1>0.7</mu1>
-        <mu2>150</mu2>
-        <fdir1 value="0 1 0" />
-        <gravity>1</gravity>
-        <kinematic>0</kinematic>
-        <enable_wind>0</enable_wind>
-        <max_contacts>10</max_contacts>
+        <selfCollide>false</selfCollide>
+        <mu1>0.7</mu1>
+        <mu2>150</mu2>
+        <fdir1 value="0 1 0" />
+        <gravity>1</gravity>
+        <maxContacts>10</maxContacts>
+        <plugin name='NuBot_Pumbaa_Gazebo_Plugin' filename='libnubot_pumbaa_plugin.so'>
+          <!--The link tags of tracks-->
+          <!-- <right_track>right_track_link</right_track> -->
+        </plugin>
       </gazebo>
     </link>
@@ -198,12 +204,14 @@
       </collision>
       <gazebo reference="rear_left_flipper_link">
-        <self_collide>false</self_collide>
-        <mu1>0.7</mu1>
-        <mu2>150</mu2>
-        <fdir1 value="0 1 0" />
-        <gravity>1</gravity>
-        <kinematic>0</kinematic>
-        <enable_wind>0</enable_wind>
-        <max_contacts>10</max_contacts>
+        <selfCollide>false</selfCollide>
+        <mu1>0.7</mu1>
+        <mu2>150</mu2>
+        <fdir1 value="0 1 0" />
+        <gravity>1</gravity>
+        <maxContacts>10</maxContacts>
+        <plugin name='NuBot_Pumbaa_Gazebo_Plugin' filename='libnubot_pumbaa_plugin.so'>
+          <!--The link tags of tracks-->
+          <!-- <left_flipper>rear_left_flipper_link</left_flipper> -->
+        </plugin>
       </gazebo>
     </link>
@@ -250,12 +258,14 @@
       </collision>
       <gazebo reference="rear_right_flipper_link">
-        <self_collide>false</self_collide>
-        <mu1>0.7</mu1>
-        <mu2>150</mu2>
-        <fdir1 value="0 1 0" />
-        <gravity>1</gravity>
-        <kinematic>0</kinematic>
-        <enable_wind>0</enable_wind>
-        <max_contacts>10</max_contacts>
+        <selfCollide>false</selfCollide>
+        <mu1>0.7</mu1>
+        <mu2>150</mu2>
+        <fdir1 value="0 1 0" />
+        <gravity>1</gravity>
+        <maxContacts>10</maxContacts>
+        <plugin name='NuBot_Pumbaa_Gazebo_Plugin' filename='libnubot_pumbaa_plugin.so'>
+          <!--The link tags of tracks-->
+          <!-- <right_flipper>rear_right_flipper_link</right_flipper> -->
+        </plugin>
       </gazebo>
     </link>
@@ -302,12 +312,14 @@
       </collision>
       <gazebo reference="front_left_flipper_link">
-        <self_collide>false</self_collide>
-        <mu1>0.7</mu1>
-        <mu2>150</mu2>
-        <fdir1 value="0 1 0" />
-        <gravity>1</gravity>
-        <kinematic>0</kinematic>
-        <enable_wind>0</enable_wind>
-        <max_contacts>10</max_contacts>
+        <selfCollide>false</selfCollide>
+        <mu1>0.7</mu1>
+        <mu2>150</mu2>
+        <fdir1 value="0 1 0" />
+        <gravity>1</gravity>
+        <maxContacts>10</maxContacts>
+        <plugin name='NuBot_Pumbaa_Gazebo_Plugin' filename='libnubot_pumbaa_plugin.so'>
+          <!--The link tags of tracks-->
+          <!-- <left_flipper>front_left_flipper_link</left_flipper> -->
+        </plugin>
       </gazebo>
     </link>
@@ -354,12 +366,14 @@
       </collision>
       <gazebo reference="front_right_flipper_link">
-        <self_collide>false</self_collide>
-        <mu1>0.7</mu1>
-        <mu2>150</mu2>
-        <fdir1 value="0 1 0" />
-        <gravity>1</gravity>
-        <kinematic>0</kinematic>
-        <enable_wind>0</enable_wind>
-        <max_contacts>10</max_contacts>
+        <selfCollide>false</selfCollide>
+        <mu1>0.7</mu1>
+        <mu2>150</mu2>
+        <fdir1 value="0 1 0" />
+        <gravity>1</gravity>
+        <maxContacts>10</maxContacts>
+        <plugin name='NuBot_Pumbaa_Gazebo_Plugin' filename='libnubot_pumbaa_plugin.so'>
+          <!--The link tags of tracks-->
+          <!-- <right_flipper>front_right_flipper_link</right_flipper> -->
+        </plugin>
       </gazebo>
     </link>

Commit message: robot & sensors in .xacro format

File: gazebo_description/models/NuBot_Pumbaa_v2/model_v2.urdf.xacro (robot description, xacro)
@@ -8,410 +8,432 @@
   <xacro:property name="track_width" value="0.18" />
   <xacro:property name="track_length" value="0.552" />
-  <xacro:property name="track_distance" value="0.14" />
+  <xacro:property name="track_distance" value="0.145" />
   <xacro:property name="flipper_radius" value="0.09" />
   <xacro:property name="flipper_width" value="0.038" />
   <xacro:property name="flipper_length" value="0.336" />
   <xacro:property name="flipper_distance" value="0.266" />
-    <!--base_link-->
-    <link name='base_link'>
-      <origin xyz="0 0 0" rpy="0 0 0" />
-      <inertial>
-        <origin xyz="0 0 0" rpy="0 0 0" />
-        <mass value="${base_mass}" />
-        <inertia ixx="0.203664" ixy="0" ixz="0"
-                 iyy="0.136197" iyz="0"
-                 izz="0.319921" />
-      </inertial>
-      <collision name='base_collision_1'>
-        <origin xyz="${track_length/2} 0 0" rpy="${PI/2} 0 0" />
-        <geometry>
-          <cylinder radius="0.07" length="0.11"/>
-        </geometry>
-      </collision>
-      <collision name='base_collision_2'>
-        <origin xyz="${-1*track_length/2} 0 0" rpy="${PI/2} 0 0" />
-        <geometry>
-          <cylinder radius="0.07" length="0.11"/>
-        </geometry>
-      </collision>
-      <collision name='base_collision'>
-        <origin xyz="0 0 0" rpy="0 0 0" />
-        <geometry>
-          <box size="${track_length} 0.11 0.14" />
-        </geometry>
-      </collision>
-      <visual name='base_visual'>
-        <origin xyz="0 0 0" rpy="0 0 0" />
-        <geometry>
-          <mesh filename="model://NuBot_Pumbaa_v2/meshes/base_link.STL" />
-        </geometry>
-      </visual>
-      <visual name='base_vive_link_visual'>
-        <origin xyz="0.16175 0 0.138" rpy="0 0 0" />
-        <geometry>
-          <mesh filename="model://NuBot_Pumbaa_v2/meshes/vive_link.STL" />
-        </geometry>
-      </visual>
-    </link>
-    <gazebo reference="base_link">
-      <selfCollide>false</selfCollide>
-      <mu1>1</mu1>
-      <mu2>1</mu2>
-      <fdir1 value="0 1 0" />
-      <gravity>1</gravity>
-      <maxContacts>10</maxContacts>
-      <plugin name='NuBot_Pumbaa_Gazebo_Plugin' filename='libnubot_pumbaa_plugin.so'>
-        <!--The link tags of tracks-->
-        <!-- <body>base_link</body> -->
-      </plugin>
-    </gazebo>
-    <!--left_track-->
-    <link name='left_track_link'>
+  <xacro:property name="flipper_visual_bias" value="0.016" />
+  <link name="base_link"></link>
+  <joint name="base_link_joint" type="fixed">
+    <origin xyz="0 0 0" rpy="0 0 0" />
+    <parent link="base_link"/>
+    <child link="chassis_link" />
+  </joint>
+  <!--chassis_link-->
+  <link name='chassis_link'>
+    <inertial>
+      <origin xyz="0 0 0" rpy="0 0 0" />
+      <mass value="${base_mass}" />
+      <inertia ixx="0.203664" ixy="0" ixz="0"
+                iyy="0.136197" iyz="0"
+                izz="0.319921" />
+    </inertial>
+    <collision name='base_collision_1'>
+      <origin xyz="${track_length/2} 0 0" rpy="${PI/2} 0 0" />
+      <geometry>
+        <cylinder radius="0.07" length="0.10"/>
+      </geometry>
+    </collision>
+    <collision name='base_collision_2'>
+      <origin xyz="${-1*track_length/2} 0 0" rpy="${PI/2} 0 0" />
+      <geometry>
+        <cylinder radius="0.07" length="0.10"/>
+      </geometry>
+    </collision>
+    <collision name='base_collision'>
+      <origin xyz="0 0 0" rpy="0 0 0" />
+      <geometry>
+        <box size="${track_length} 0.10 0.14" />
+      </geometry>
+    </collision>
+    <visual name='base_visual'>
+      <origin xyz="0 0 0" rpy="0 0 0" />
+      <geometry>
+        <mesh filename="model://NuBot_Pumbaa_v2/meshes/base_link.STL" />
+      </geometry>
+    </visual>
+    <visual name='base_vive_link_visual'>
+      <origin xyz="0.16175 0 0.138" rpy="0 0 0" />
+      <geometry>
+        <mesh filename="model://NuBot_Pumbaa_v2/meshes/vive_link.STL" />
+      </geometry>
+    </visual>
+  </link>
+  <gazebo reference="chassis_link">
+    <selfCollide>false</selfCollide>
+    <mu1>1</mu1>
+    <mu2>1</mu2>
+    <fdir1 value="0 1 0" />
+    <gravity>1</gravity>
+    <maxContacts>10</maxContacts>
+  </gazebo>
+  <!--left_track-->
+  <link name='left_track_link'>
+    <inertial>
+      <origin xyz="0 0 0" rpy="0 0 0" />
+      <mass value="${track_mass}" />
+      <inertia ixx="0.15" ixy="0" ixz="0"
+                iyy="0.9" iyz="0"
+                izz="0.9" />
+    </inertial>
+    <visual name='left_track_visual'>
+      <origin xyz="0 ${-1*track_distance} 0" rpy="0 0 0" />
+      <geometry>
+        <mesh filename="model://NuBot_Pumbaa_v2/meshes/left_track_link.STL" />
+      </geometry>
+    </visual>
+    <collision name='left_track_collision_1'>
+      <origin xyz="${track_length/2} 0 0" rpy="${PI/2} 0 0" />
+      <geometry>
+        <cylinder radius="${track_radius}" length="${track_width}"/>
+      </geometry>
+    </collision>
+    <collision name='left_track_collision_2'>
+      <origin xyz="${-1*track_length/2} 0 0" rpy="${PI/2} 0 0" />
+      <geometry>
+        <cylinder radius="${track_radius}" length="${track_width}"/>
+      </geometry>
+    </collision>
+    <collision name='left_track_collision'>
+      <origin xyz="0 0 0" rpy="0 0 0" />
+      <geometry>
+        <box size="${track_length} ${track_width} ${track_radius*2}" />
+      </geometry>
+    </collision>
+  </link>
+  <gazebo reference="left_track_link">
+    <selfCollide>false</selfCollide>
+    <mu1>0.7</mu1>
+    <mu2>150</mu2>
+    <fdir1 value="0 1 0" />
+    <gravity>1</gravity>
+    <maxContacts>10</maxContacts>
+  </gazebo>
+  <!--left_track joints-->
+  <joint name='left_track_joint' type='revolute'><!-- fixed -->
+    <origin xyz="0 ${track_distance} 0" rpy="0 0 0" />
+    <child link="left_track_link" />
+    <parent link="chassis_link" />
+    <limit lower="-1e-16" upper="1e-16" effort="10000" velocity="10000"/>
+    <axis xyz="0 0 0"/>
+    <dynamics damping="10000" friction="10000"/>
+  </joint>
+  <!--right_track-->
+  <link name='right_track_link'>
+    <inertial>
+      <origin xyz="0 0 0" rpy="0 0 0" />
+      <mass value="${track_mass}" />
+      <inertia ixx="0.15" ixy="0" ixz="0"
+                iyy="0.9" iyz="0"
+                izz="0.9" />
+    </inertial>
+    <visual name='right_track_visual'>
       <origin xyz="0 ${track_distance} 0" rpy="0 0 0" />
-      <inertial>
-        <origin xyz="0 0 0" rpy="0 0 0" />
-        <mass value="${track_mass}" />
-        <inertia ixx="0.15" ixy="0" ixz="0"
-                 iyy="0.9" iyz="0"
-                 izz="0.9" />
-      </inertial>
-      <visual name='left_track_visual'>
-        <origin xyz="0 ${-1*track_distance} 0" rpy="0 0 0" />
-        <geometry>
-          <mesh filename="model://NuBot_Pumbaa_v2/meshes/left_track_link.STL" />
-        </geometry>>
-      </visual>
-      <collision name='left_track_collision_1'>
-        <origin xyz="${track_length/2} 0 0" rpy="${PI/2} 0 0" />
-        <geometry>
-          <cylinder radius="${track_radius}" length="${track_width}"/>
-        </geometry>
-      </collision>
-      <collision name='left_track_collision_2'>
-        <origin xyz="${-1*track_length/2} 0 0" rpy="${PI/2} 0 0" />
-        <geometry>
-          <cylinder radius="${track_radius}" length="${track_width}"/>
-        </geometry>
-      </collision>
-      <collision name='left_track_collision'>
-        <origin xyz="0 0 0" rpy="0 0 0" />
-        <geometry>
-          <box size="${track_length} ${track_width} ${track_radius*2}" />
-        </geometry>
-      </collision>
-      <gazebo reference="left_track_link">
-        <selfCollide>false</selfCollide>
-        <mu1>0.7</mu1>
-        <mu2>150</mu2>
-        <fdir1 value="0 1 0" />
-        <gravity>1</gravity>
-        <maxContacts>10</maxContacts>
-        <plugin name='NuBot_Pumbaa_Gazebo_Plugin' filename='libnubot_pumbaa_plugin.so'>
-          <!--The link tags of tracks-->
-          <!-- <left_track>left_track_link</left_track> -->
-        </plugin>
-      </gazebo>
-    </link>
-    <!--right_track-->
-    <link name='right_track_link'>
-      <origin xyz="0 ${-1*track_distance} 0" rpy="0 0 0" />
-      <inertial>
-        <origin xyz="0 0 0" rpy="0 0 0" />
-        <mass value="${track_mass}" />
-        <inertia ixx="0.15" ixy="0" ixz="0"
-                 iyy="0.9" iyz="0"
-                 izz="0.9" />
-      </inertial>
-      <visual name='right_track_visual'>
-        <origin xyz="0 ${track_distance} 0" rpy="0 0 0" />
-        <geometry>
-          <mesh filename="model://NuBot_Pumbaa_v2/meshes/right_track_link.STL" />
-        </geometry>>
-      </visual>
-      <collision name='right_track_collision_1'>
-        <origin xyz="${track_length/2} 0 0" rpy="${PI/2} 0 0" />
-        <geometry>
-          <cylinder radius="${track_radius}" length="${track_width}"/>
-        </geometry>
-      </collision>
-      <collision name='right_track_collision_2'>
-        <origin xyz="${-1*track_length/2} 0 0" rpy="${PI/2} 0 0" />
-        <geometry>
-          <cylinder radius="${track_radius}" length="${track_width}"/>
-        </geometry>
-      </collision>
-      <collision name='right_track_collision'>
-        <origin xyz="0 0 0" rpy="0 0 0" />
-        <geometry>
-          <box size="${track_length} ${track_width} ${track_radius*2}" />
-        </geometry>
-      </collision>
-      <gazebo reference="right_track_link">
-        <selfCollide>false</selfCollide>
-        <mu1>0.7</mu1>
-        <mu2>150</mu2>
-        <fdir1 value="0 1 0" />
-        <gravity>1</gravity>
-        <maxContacts>10</maxContacts>
-        <plugin name='NuBot_Pumbaa_Gazebo_Plugin' filename='libnubot_pumbaa_plugin.so'>
-          <!--The link tags of tracks-->
-          <!-- <right_track>right_track_link</right_track> -->
-        </plugin>
-      </gazebo>
-    </link>
-    <!--main_track joints-->
-    <joint name='left_track_joint' type='fixed'>
-      <parent link="base_link" />
-      <child link="left_track_link" />
-    </joint>
-    <joint name='right_track_joint' type='fixed'>
-      <parent link="base_link" />
-      <child link="right_track_link" />
-    </joint>
-    <!--rear_left_flipper-->
-    <link name='rear_left_flipper_link'>
-      <origin xyz="${-1*track_length/2} ${flipper_distance} 0" rpy="0 0 0" />
-      <inertial>
-        <origin xyz="${-1*flipper_length/2} 0 0" rpy="0 0 0" />
-        <mass value="${flipper_mass}" />
-        <inertia ixx="0.0025" ixy="0" ixz="0"
-                 iyy="0.022" iyz="0"
-                 izz="0.02" />
-      </inertial>
-      <visual name='rear_left_flipper_visual'>
-        <origin xyz="0 0 0" rpy="0 0 0" />
-        <geometry>
-          <mesh filename="model://NuBot_Pumbaa_v2/meshes/back_left_fin_link.STL" />
-        </geometry>>
-      </visual>
-      <collision name='rear_left_flipper_collision_large_wheel_collision'>
-        <origin xyz="0 0 0" rpy="${PI/2} 0 0" />
-        <geometry>
-          <cylinder radius="${flipper_radius}" length="${flipper_width}"/>
-        </geometry>
-      </collision>
-      <collision name='rear_left_flipper_collision_small_wheel_collision'>
-        <origin xyz="${-1*flipper_length} 0 0" rpy="${PI/2} 0 0" />
-        <geometry>
-          <cylinder radius="${flipper_radius}" length="${flipper_width}"/>
-        </geometry>
-      </collision>
-      <collision name='rear_left_flipper_collision_middle_bar_collision'>
-        <origin xyz="${-1*flipper_length/2} 0 0" rpy="0 0 0" />
-        <geometry>
-          <box size="${flipper_length} ${flipper_width} ${flipper_radius*2}" />
-        </geometry>
-      </collision>
-      <gazebo reference="rear_left_flipper_link">
-        <selfCollide>false</selfCollide>
-        <mu1>0.7</mu1>
-        <mu2>150</mu2>
-        <fdir1 value="0 1 0" />
-        <gravity>1</gravity>
-        <maxContacts>10</maxContacts>
-        <plugin name='NuBot_Pumbaa_Gazebo_Plugin' filename='libnubot_pumbaa_plugin.so'>
-          <!--The link tags of tracks-->
-          <!-- <left_flipper>rear_left_flipper_link</left_flipper> -->
-        </plugin>
-      </gazebo>
-    </link>
-    <joint name='rear_left_flipper_joint' type='revolute'>
-      <child link="rear_left_flipper_link" />
-      <parent link="base_link" />
-      <origin xyz="0 0 0" rpy="0 0 0" />
-      <axis xyz="0 1 0" />
-      <limit lower="-3" upper="3" effort="-1" velocity="0.3" />
-    </joint>
-    <!--rear_right_flipper-->
-    <link name='rear_right_flipper_link'>
-      <origin xyz="${-1*track_length/2} ${-1*flipper_distance} 0" rpy="0 0 0" />
-      <inertial>
-        <origin xyz="${-1*flipper_length/2} 0 0" rpy="0 0 0" />
-        <mass value="${flipper_mass}" />
-        <inertia ixx="0.0025" ixy="0" ixz="0"
-                 iyy="0.022" iyz="0"
-                 izz="0.02" />
-      </inertial>
-      <visual name='rear_right_flipper_visual'>
-        <origin xyz="0 0 0" rpy="0 0 0" />
-        <geometry>
-          <mesh filename="model://NuBot_Pumbaa_v2/meshes/back_right_fin_link.STL" />
-        </geometry>>
-      </visual>
-      <collision name='rear_right_flipper_collision_large_wheel_collision'>
-        <origin xyz="0 0 0" rpy="${PI/2} 0 0" />
-        <geometry>
-          <cylinder radius="${flipper_radius}" length="${flipper_width}"/>
-        </geometry>
-      </collision>
-      <collision name='rear_right_flipper_collision_small_wheel_collision'>
-        <origin xyz="${-1*flipper_length} 0 0" rpy="${PI/2} 0 0" />
-        <geometry>
-          <cylinder radius="${flipper_radius}" length="${flipper_width}"/>
-        </geometry>
-      </collision>
-      <collision name='rear_right_flipper_collision_middle_bar_collision'>
-        <origin xyz="${-1*flipper_length/2} 0 0" rpy="0 0 ${PI}" />
-        <geometry>
-          <box size="${flipper_length} ${flipper_width} ${flipper_radius*2}" />
-        </geometry>
-      </collision>
-      <gazebo reference="rear_right_flipper_link">
-        <selfCollide>false</selfCollide>
-        <mu1>0.7</mu1>
-        <mu2>150</mu2>
-        <fdir1 value="0 1 0" />
-        <gravity>1</gravity>
-        <maxContacts>10</maxContacts>
-        <plugin name='NuBot_Pumbaa_Gazebo_Plugin' filename='libnubot_pumbaa_plugin.so'>
-          <!--The link tags of tracks-->
-          <!-- <right_flipper>rear_right_flipper_link</right_flipper> -->
-        </plugin>
-      </gazebo>
-    </link>
-    <joint name='rear_right_flipper_joint' type='revolute'>
-      <child link="rear_right_flipper_link" />
-      <parent link="base_link" />
-      <origin xyz="0 0 0" rpy="0 0 0" />
-      <axis xyz="0 1 0" />
-      <limit lower="-3" upper="3" effort="-1" velocity="0.3" />
-    </joint>
-    <!--front_left_flipper-->
-    <link name='front_left_flipper_link'>
-      <origin xyz="${track_length/2} ${flipper_distance} 0" rpy="0 0 0" />
-      <inertial>
-        <origin xyz="${flipper_length/2} 0 0" rpy="0 0 0" />
-        <mass value="${flipper_mass}" />
-        <inertia ixx="0.0025" ixy="0" ixz="0"
-                 iyy="0.022" iyz="0"
-                 izz="0.02" />
-      </inertial>
-      <visual name='front_left_flipper_visual'>
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
File: gazebo_description/models/RS_Helios_5515/model.urdf.xacro (robot description, xacro)
@@ -2,5 +2,4 @@
 <robot xmlns:xacro="http://www.ros.org/wiki/xacro" name="RS_Helios_5515">
     <link name='base_link'>
-      <origin rpy="0 0 0" xyz="0 0 0"/>
       <inertial>
         <origin rpy="0 0 0" xyz="0 0 0"/>
