Commit message: .xacro sensor visualize bug fixed, adjust patameters

File: gazebo_description/models/NuBot_Pumbaa_v2/model_v2.urdf.xacro (robot description, xacro)
@@ -390,5 +390,5 @@
       <flip_initial>1.5708</flip_initial>
       <!--The parameters of tracks-->
-      <tracksSeparation>0.285</tracksSeparation>
+      <tracksSeparation>0.29</tracksSeparation>
       <steeringEfficiency>0.5</steeringEfficiency>
       <maxLinearSpeed>2.0</maxLinearSpeed>
@@ -398,8 +398,9 @@
   <!-- IMU -->
   <link name="imu_link">
-    <inertial>
+    <!-- <inertial>
       <mass value="0.1"/>
-    </inertial>
+    </inertial> -->
     <visual name='imu_visual'>
+      <origin xyz="0 0 0.015" rpy="0 0 0"/>
       <geometry>
         <box size="0.05 0.04 0.03" />
@@ -407,5 +408,5 @@
     </visual>
     <collision name='imu_collision'>
-      <origin rpy="0 0 0" xyz="0 0 0"/>
+      <origin xyz="0 0 0.015" rpy="0 0 0"/>
       <geometry>
         <box size="0.05 0.04 0.03" />
@@ -413,6 +414,7 @@
     </collision>
   </link>
-  <joint name="imu_link_joint" type="fixed">
-    <origin xyz="-0.16175 0 0.14" rpy="0 0 ${PI}" />
+  <joint name="imu_link_joint" type='fixed'>
+    <origin xyz="-0.22175 0 0.131" rpy="0 0 ${PI}" />
+    <!--0.16175+0.06=0.22175 0.118+0.013=0.131-->
     <parent link="chassis_link"/>
     <child link="imu_link" />
@@ -432,8 +434,13 @@
     </plugin>
   </gazebo>
-  <!-- RS-Helios includes -->
+  <!-- RS-Helios includes --><!--0.16175+0.06=0.22175 0.118+0.073+0.0635=0.2545-->
   <xacro:include filename="$(find gazebo_description)/models/RS_Helios_5515/model_2.urdf.xacro"/>
-  <xacro:RS_Helios_5515 parent="chassis_link" name="re_helios" topic="/lidar_points" hz="10" samples="1800" min_angle="-${PI/2}" max_angle="${PI/2}" min_range ="0.2" max_range="50.0" gpu="false">
-    <origin xyz="-0.21175 0 0.224" rpy="0 0 ${PI}" />
+  <xacro:RS_Helios_5515 parent="chassis_link" name="rs_helios" topic="/lidar_points" hz="10" samples="1800" min_angle="-${PI/2}" max_angle="${PI/2}" min_range ="0.2" max_range="50.0" gpu="false">
+    <origin xyz="-0.22175 0 0.2545" rpy="0 0 ${PI}" />
   </xacro:RS_Helios_5515>
+  <!-- RS-Bpearl includes --><!--0.16175+0.06=0.22175 0.118+0.073+0.0635=0.2545-->
+  <!-- <xacro:include filename="$(find gazebo_description)/models/RS_Bpearl/model_2.urdf.xacro"/>
+  <xacro:RS_Bpearl parent="chassis_link" name="rs_bpearl" topic="/lidar_points" hz="10" lasers="32" samples="1800" min_angle="-${PI/2}" max_angle="${PI/2}" min_range ="0.1" max_range="50.0" gpu="true">
+    <origin xyz="-0.34175 0 0.2045" rpy="0 ${PI/2} 0" />
+  </xacro:RS_Bpearl> -->
 </robot>

File: gazebo_description/models/RS_Bpearl/model.urdf.xacro (robot description, xacro)
@@ -2,7 +2,6 @@
 <robot xmlns:xacro="http://www.ros.org/wiki/xacro" name="RS_Bpearl">
     <link name='base_link'>
-      <origin rpy="0 0 0" xyz="0 0 0"/>
       <inertial>
-        <origin xyz="0 -0.00079641 0.026317"/>
+        <origin xyz="0 -0.00079641 0.026317" rpy="0 0 0"/>
         <mass value="0.92"/>
         <inertia>
@@ -13,5 +12,5 @@
       </inertial>
       <collision name='collision'>
-        <origin xyz="0 0 0.04"/>
+        <origin xyz="0 0 0.04" rpy="0 0 0"/>
         <geometry>
           <cylinder radius="0.05" length="0.11"/>
@@ -20,5 +19,5 @@
       </collision>
       <visual name='visual'>
-        <origin rpy="0 0 0" xyz="0 0 0"/>
+        <origin xyz="0 0 0" rpy="0 0 0"/>
         <geometry>
           <mesh filename="model://RS_Bpearl/meshes/RS_Bpearl_frame.STL" />

File: gazebo_description/models/RS_Bpearl/model_2.urdf.xacro (robot description, xacro)
@@ -1,6 +1,6 @@
 <?xml version="1.0"?>
-<robot xmlns:xacro="http://www.ros.org/wiki/xacro" name="RS_Helios_5515">
+<robot xmlns:xacro="http://www.ros.org/wiki/xacro" name="RS_Bpearl">
   <xacro:property name="M_PI" value="3.1415926535897931" />
-  <xacro:macro name="RS_Helios_5515" params="*origin parent:=base_link name:=rs_helios topic:=/lidar_points organize_cloud:=false hz:=10 lasers:=32 samples:=2187 collision_range:=0.2 min_range:=0.2 max_range:=100.0 noise:=0.008 min_angle:=-${M_PI} max_angle:=${M_PI} gpu:=false">
+  <xacro:macro name="RS_Bpearl" params="*origin parent:=base_link name:=rs_bpearl topic:=/lidar_points organize_cloud:=false hz:=10 lasers:=32 samples:=2187 collision_range:=0.1 min_range:=0.1 max_range:=100.0 noise:=0.008 min_angle:=-${M_PI} max_angle:=${M_PI} gpu:=false">
     <joint name="${name}_base_mount_joint" type="fixed">
       <xacro:insert_block name="origin" />
@@ -8,16 +8,16 @@
       <child link="${name}_base_link"/>
     </joint>
-    <link name="${name}_base_link">
+    <link name='${name}_base_link'>
       <!-- <inertial>
-        <origin xyz="0 0 0" rpy="0 0 0"/>
-        <mass value="0.9"/>
+        <origin xyz="0 -0.00079641 0.026317" rpy="0 0 0"/>
+        <mass value="0.92"/>
         <inertia>
-        <inertia ixx="0.0025413" ixy="0" ixz="0"
-                  iyy="0.0016941" iyz="0"
-                  izz="0.0024448"/>
+        <inertia ixx="0.0015364" ixy="0" ixz="0"
+                  iyy="0.0014894" iyz="0"
+                  izz="0.0016331"/>
         </inertia>
       </inertial> -->
       <collision name='collision'>
-        <origin xyz="0 0 -0.02" rpy="0 0 0"/>
+        <origin xyz="0 0 0.04" rpy="0 0 0"/>
         <geometry>
           <cylinder radius="0.05" length="0.11"/>
@@ -28,5 +28,5 @@
         <origin xyz="0 0 0" rpy="0 0 0"/>
         <geometry>
-          <mesh filename="model://RS_Helios_5515/meshes/RS_Helios_frame.STL" />
+          <mesh filename="model://RS_Bpearl/meshes/RS_Bpearl_frame.STL" />
         </geometry>
       </visual>
@@ -41,7 +41,7 @@
     <gazebo reference="${name}">
       <xacro:if value="${gpu}">
-        <sensor type="gpu_ray" name="${name}-RS_Helios_5515">
+        <sensor type="gpu_ray" name="${name}-RS_Bpearl">
           <pose>0 0 0 0 0 0</pose>
-          <visualize>false</visualize>
+          <visualize>true</visualize>
           <update_rate>${hz}</update_rate>
           <ray>
@@ -56,6 +56,6 @@
                 <samples>${lasers}</samples>
                 <resolution>1</resolution>
-                <min_angle>-${55*M_PI/180.0}</min_angle>
-                <max_angle> ${15*M_PI/180.0}</max_angle>
+                <min_angle>-${84*M_PI/180.0}</min_angle>
+                <max_angle>-${2.3125*M_PI/180.0}</max_angle>
               </vertical>
             </scan>
@@ -82,5 +82,5 @@
       </xacro:if>
       <xacro:unless value="${gpu}">
-        <sensor type="ray" name="${name}-RS_Helios_5515">
+        <sensor type="ray" name="${name}-RS_Bpearl">
           <pose>0 0 0 0 0 0</pose>
           <visualize>false</visualize>
@@ -97,6 +97,6 @@
                 <samples>${lasers}</samples>
                 <resolution>1</resolution>
-                <min_angle>-${55*M_PI/180.0}</min_angle>
-                <max_angle> ${15*M_PI/180.0}</max_angle>
+                <min_angle>-${89.5*M_PI/180.0}</min_angle>
+                <max_angle>-${2.3125*M_PI/180.0}</max_angle>
               </vertical>
             </scan>

File: gazebo_description/models/RS_Helios_5515/model.urdf.xacro (robot description, xacro)
@@ -3,5 +3,5 @@
     <link name='base_link'>
       <inertial>
-        <origin rpy="0 0 0" xyz="0 0 0"/>
+        <origin xyz="0 0 0" rpy="0 0 0"/>
         <mass value="0.9"/>
         <inertia>
@@ -12,5 +12,5 @@
       </inertial>
       <collision name='collision'>
-        <origin xyz="0 0 -0.02"/>
+        <origin xyz="0 0 -0.02" rpy="0 0 0"/>
         <geometry>
           <cylinder radius="0.05" length="0.11"/>
@@ -19,5 +19,5 @@
       </collision>
       <visual name='visual'>
-        <origin rpy="0 0 0" xyz="0 0 0"/>
+        <origin xyz="0 0 0" rpy="0 0 0"/>
         <geometry>
           <mesh filename="model://RS_Helios_5515/meshes/RS_Helios_frame.STL" />

Commit message: adjust parameters of sensors

File: gazebo_description/models/NuBot_Pumbaa_v2/model_v2.urdf.xacro (robot description, xacro)
@@ -396,51 +396,23 @@
     </plugin>
   </gazebo>
-  <!-- IMU -->
-  <link name="imu_link">
-    <!-- <inertial>
-      <mass value="0.1"/>
-    </inertial> -->
-    <visual name='imu_visual'>
-      <origin xyz="0 0 0.015" rpy="0 0 0"/>
-      <geometry>
-        <box size="0.05 0.04 0.03" />
-      </geometry>
-    </visual>
-    <collision name='imu_collision'>
-      <origin xyz="0 0 0.015" rpy="0 0 0"/>
-      <geometry>
-        <box size="0.05 0.04 0.03" />
-      </geometry>
-    </collision>
-  </link>
-  <joint name="imu_link_joint" type='fixed'>
-    <origin xyz="-0.22175 0 0.131" rpy="0 0 ${PI}" />
-    <!--0.16175+0.06=0.22175 0.118+0.013=0.131-->
-    <parent link="chassis_link"/>
-    <child link="imu_link" />
-  </joint>
-  <gazebo>
-    <plugin name="imu_controller" filename="libhector_gazebo_ros_imu.so">
-      <robotNamespace>/</robotNamespace>
-      <updateRate>400.0</updateRate>
-      <bodyName>imu_link</bodyName>
-      <topicName>imu/data</topicName>
-      <accelDrift>0.005 0.005 0.005</accelDrift>
-      <accelGaussianNoise>0.005 0.005 0.005</accelGaussianNoise>
-      <rateDrift>0.005 0.005 0.005 </rateDrift>
-      <rateGaussianNoise>0.005 0.005 0.005 </rateGaussianNoise>
-      <headingDrift>0.005</headingDrift>
-      <headingGaussianNoise>0.005</headingGaussianNoise>
-    </plugin>
-  </gazebo>
-  <!-- RS-Helios includes --><!--0.16175+0.06=0.22175 0.118+0.073+0.0635=0.2545-->
-  <xacro:include filename="$(find gazebo_description)/models/RS_Helios_5515/model_2.urdf.xacro"/>
-  <xacro:RS_Helios_5515 parent="chassis_link" name="rs_helios" topic="/lidar_points" hz="10" samples="1800" min_angle="-${PI/2}" max_angle="${PI/2}" min_range ="0.2" max_range="50.0" gpu="false">
-    <origin xyz="-0.22175 0 0.2545" rpy="0 0 ${PI}" />
-  </xacro:RS_Helios_5515>
-  <!-- RS-Bpearl includes --><!--0.16175+0.06=0.22175 0.118+0.073+0.0635=0.2545-->
-  <!-- <xacro:include filename="$(find gazebo_description)/models/RS_Bpearl/model_2.urdf.xacro"/>
-  <xacro:RS_Bpearl parent="chassis_link" name="rs_bpearl" topic="/lidar_points" hz="10" lasers="32" samples="1800" min_angle="-${PI/2}" max_angle="${PI/2}" min_range ="0.1" max_range="50.0" gpu="true">
-    <origin xyz="-0.34175 0 0.2045" rpy="0 ${PI/2} 0" />
-  </xacro:RS_Bpearl> -->
+  <!-- RS-Helios includes -->
+  <!-- <xacro:include filename="$(find gazebo_description)/models/RS_Helios_5515/model_2.urdf.xacro"/>
+  <xacro:RS_Helios_5515 parent="chassis_link" name="rs_helios" topic="/lidar_points" hz="10" samples="900" min_angle="-${PI/2}" max_angle="${PI/2}" min_range ="0.2" max_range="50.0" gpu="false">
+    <origin xyz="-0.221 0 0.2545" rpy="0 0 ${PI}" />
+  </xacro:RS_Helios_5515> -->
+  <!-- IMU includes (RS-Helios) -->
+  <!-- <xacro:include filename="$(find gazebo_description)/models/IMU/model.urdf.xacro"/>
+  <xacro:IMU parent="chassis_link" name="imu" topic="/imu/data" hz="400">
+    <origin xyz="-0.221 0 0.131" rpy="0 0 ${PI}" />
+  </xacro:IMU> -->
+  <!-- RS-Bpearl includes -->
+  <xacro:include filename="$(find gazebo_description)/models/RS_Bpearl/model_2.urdf.xacro"/>
+  <xacro:RS_Bpearl parent="chassis_link" name="rs_bpearl" topic="/velodyne_points" hz="10" lasers="32" samples="1800" min_angle="-${PI}" max_angle="${PI}" min_range ="0.1" max_range="50.0" gpu="true">
+    <origin xyz="-0.36277 0 0.2115" rpy="0 ${PI/2} 0" />
+  </xacro:RS_Bpearl>
+  <!-- IMU includes (RS-Bpearl) -->
+  <xacro:include filename="$(find gazebo_description)/models/IMU/model.urdf.xacro"/>
+  <xacro:IMU parent="chassis_link" name="imu" topic="/imu/data" hz="400">
+    <origin xyz="-0.3185 0 0.133" rpy="0 0 ${PI}" />
+  </xacro:IMU>
 </robot>

File: gazebo_description/models/RS_Bpearl/model_2.urdf.xacro (robot description, xacro)
@@ -3,10 +3,10 @@
   <xacro:property name="M_PI" value="3.1415926535897931" />
   <xacro:macro name="RS_Bpearl" params="*origin parent:=base_link name:=rs_bpearl topic:=/lidar_points organize_cloud:=false hz:=10 lasers:=32 samples:=2187 collision_range:=0.1 min_range:=0.1 max_range:=100.0 noise:=0.008 min_angle:=-${M_PI} max_angle:=${M_PI} gpu:=false">
-    <joint name="${name}_base_mount_joint" type="fixed">
+    <joint name="${name}_mount_joint" type="fixed">
       <xacro:insert_block name="origin" />
       <parent link="${parent}"/>
-      <child link="${name}_base_link"/>
+      <child link="${name}_link"/>
     </joint>
-    <link name='${name}_base_link'>
+    <link name='${name}_link'>
       <!-- <inertial>
         <origin xyz="0 -0.00079641 0.026317" rpy="0 0 0"/>
@@ -32,12 +32,6 @@
       </visual>
     </link>
-    <joint name="${name}_base_scan_joint" type="fixed" >
-      <origin xyz="0 0 0" rpy="0 0 0" />
-      <parent link="${name}_base_link" />
-      <child link="${name}"/>
-    </joint>
-    <link name="${name}"/>
     <!-- Gazebo requires the velodyne_gazebo_plugins package -->
-    <gazebo reference="${name}">
+    <gazebo reference="${name}_link">
       <xacro:if value="${gpu}">
         <sensor type="gpu_ray" name="${name}-RS_Bpearl">
@@ -56,5 +50,5 @@
                 <samples>${lasers}</samples>
                 <resolution>1</resolution>
-                <min_angle>-${84*M_PI/180.0}</min_angle>
+                <min_angle>-${84.9*M_PI/180.0}</min_angle>
                 <max_angle>-${2.3125*M_PI/180.0}</max_angle>
               </vertical>
@@ -73,5 +67,5 @@
           <plugin name="gazebo_ros_laser_controller" filename="libgazebo_ros_velodyne_gpu_laser.so">
             <topicName>${topic}</topicName>
-            <frameName>${name}</frameName>
+            <frameName>${name}_link</frameName>
             <organize_cloud>${organize_cloud}</organize_cloud>
             <min_range>${min_range}</min_range>
@@ -114,5 +108,5 @@
           <plugin name="gazebo_ros_laser_controller" filename="libgazebo_ros_velodyne_laser.so">
             <topicName>${topic}</topicName>
-            <frameName>${name}</frameName>
+            <frameName>${name}_link</frameName>
             <organize_cloud>${organize_cloud}</organize_cloud>
             <min_range>${min_range}</min_range>

File: gazebo_description/models/RS_Helios_5515/model_2.urdf.xacro (robot description, xacro)
@@ -3,10 +3,10 @@
   <xacro:property name="M_PI" value="3.1415926535897931" />
   <xacro:macro name="RS_Helios_5515" params="*origin parent:=base_link name:=rs_helios topic:=/lidar_points organize_cloud:=false hz:=10 lasers:=32 samples:=2187 collision_range:=0.2 min_range:=0.2 max_range:=100.0 noise:=0.008 min_angle:=-${M_PI} max_angle:=${M_PI} gpu:=false">
-    <joint name="${name}_base_mount_joint" type="fixed">
+    <joint name="${name}_mount_joint" type="fixed">
       <xacro:insert_block name="origin" />
       <parent link="${parent}"/>
-      <child link="${name}_base_link"/>
+      <child link="${name}_link"/>
     </joint>
-    <link name="${name}_base_link">
+    <link name="${name}_link">
       <!-- <inertial>
         <origin xyz="0 0 0" rpy="0 0 0"/>
@@ -32,12 +32,6 @@
       </visual>
     </link>
-    <joint name="${name}_base_scan_joint" type="fixed" >
-      <origin xyz="0 0 0" rpy="0 0 0" />
-      <parent link="${name}_base_link" />
-      <child link="${name}"/>
-    </joint>
-    <link name="${name}"/>
     <!-- Gazebo requires the velodyne_gazebo_plugins package -->
-    <gazebo reference="${name}">
+    <gazebo reference="${name}_link">
       <xacro:if value="${gpu}">
         <sensor type="gpu_ray" name="${name}-RS_Helios_5515">
@@ -73,5 +67,5 @@
           <plugin name="gazebo_ros_laser_controller" filename="libgazebo_ros_velodyne_gpu_laser.so">
             <topicName>${topic}</topicName>
-            <frameName>${name}</frameName>
+            <frameName>${name}_link</frameName>
             <organize_cloud>${organize_cloud}</organize_cloud>
             <min_range>${min_range}</min_range>
@@ -114,5 +108,5 @@
           <plugin name="gazebo_ros_laser_controller" filename="libgazebo_ros_velodyne_laser.so">
             <topicName>${topic}</topicName>
-            <frameName>${name}</frameName>
+            <frameName>${name}_link</frameName>
             <organize_cloud>${organize_cloud}</organize_cloud>
             <min_range>${min_range}</min_range>

Commit message: bpearl lidar parameters fix

File: gazebo_description/models/NuBot_Pumbaa_v2/model_v2.urdf.xacro (robot description, xacro)
@@ -397,22 +397,22 @@
   </gazebo>
   <!-- RS-Helios includes -->
-  <!-- <xacro:include filename="$(find gazebo_description)/models/RS_Helios_5515/model_2.urdf.xacro"/>
-  <xacro:RS_Helios_5515 parent="chassis_link" name="rs_helios" topic="/lidar_points" hz="10" samples="900" min_angle="-${PI/2}" max_angle="${PI/2}" min_range ="0.2" max_range="50.0" gpu="false">
+  <xacro:include filename="$(find gazebo_description)/models/RS_Helios_5515/model_2.urdf.xacro"/>
+  <xacro:RS_Helios_5515 parent="chassis_link" name="rs_helios" topic="/lidar_points" hz="10" samples="1800" min_angle="-${PI}" max_angle="${PI}" min_range ="0.2" max_range="50.0" gpu="true">
     <origin xyz="-0.221 0 0.2545" rpy="0 0 ${PI}" />
-  </xacro:RS_Helios_5515> -->
+  </xacro:RS_Helios_5515>
   <!-- IMU includes (RS-Helios) -->
+  <xacro:include filename="$(find gazebo_description)/models/IMU/model.urdf.xacro"/>
+  <xacro:IMU parent="chassis_link" name="imu" topic="/imu/data" hz="400">
+    <origin xyz="-0.221 0 0.131" rpy="0 0 ${PI}" />
+  </xacro:IMU>
+  <!-- RS-Bpearl includes -->
+  <!-- <xacro:include filename="$(find gazebo_description)/models/RS_Bpearl/model_2.urdf.xacro"/>
+  <xacro:RS_Bpearl parent="chassis_link" name="rs_bpearl" topic="/lidar_points" hz="10" lasers="32" samples="1800" min_angle="-${PI}" max_angle="${PI}" min_range ="0.1" max_range="50.0" gpu="true">
+    <origin xyz="-0.36277 0 0.2115" rpy="${PI} ${PI/2} 0" />
+  </xacro:RS_Bpearl> -->
+  <!-- IMU includes (RS-Bpearl) -->
   <!-- <xacro:include filename="$(find gazebo_description)/models/IMU/model.urdf.xacro"/>
   <xacro:IMU parent="chassis_link" name="imu" topic="/imu/data" hz="400">
-    <origin xyz="-0.221 0 0.131" rpy="0 0 ${PI}" />
+    <origin xyz="-0.3185 0 0.133" rpy="0 0 ${PI}" />
   </xacro:IMU> -->
-  <!-- RS-Bpearl includes -->
-  <xacro:include filename="$(find gazebo_description)/models/RS_Bpearl/model_2.urdf.xacro"/>
-  <xacro:RS_Bpearl parent="chassis_link" name="rs_bpearl" topic="/velodyne_points" hz="10" lasers="32" samples="1800" min_angle="-${PI}" max_angle="${PI}" min_range ="0.1" max_range="50.0" gpu="true">
-    <origin xyz="-0.36277 0 0.2115" rpy="0 ${PI/2} 0" />
-  </xacro:RS_Bpearl>
-  <!-- IMU includes (RS-Bpearl) -->
-  <xacro:include filename="$(find gazebo_description)/models/IMU/model.urdf.xacro"/>
-  <xacro:IMU parent="chassis_link" name="imu" topic="/imu/data" hz="400">
-    <origin xyz="-0.3185 0 0.133" rpy="0 0 ${PI}" />
-  </xacro:IMU>
 </robot>

File: gazebo_description/models/RS_Bpearl/model_2.urdf.xacro (robot description, xacro)
@@ -19,5 +19,5 @@
       </inertial> -->
       <collision name='collision'>
-        <origin xyz="0 0 0.04" rpy="0 0 0"/>
+        <origin xyz="0 0 -0.04" rpy="0 0 0"/>
         <geometry>
           <cylinder radius="0.05" length="0.11"/>
@@ -26,5 +26,5 @@
       </collision>
       <visual name='visual'>
-        <origin xyz="0 0 0" rpy="0 0 0"/>
+        <origin xyz="0 0 0" rpy="${M_PI} 0 0"/>
         <geometry>
           <mesh filename="model://RS_Bpearl/meshes/RS_Bpearl_frame.STL" />
@@ -50,6 +50,6 @@
                 <samples>${lasers}</samples>
                 <resolution>1</resolution>
-                <min_angle>-${84.9*M_PI/180.0}</min_angle>
-                <max_angle>-${2.3125*M_PI/180.0}</max_angle>
+                <min_angle>${2.3125*M_PI/180.0}</min_angle>
+                <max_angle>${84.9*M_PI/180.0}</max_angle>
               </vertical>
             </scan>
@@ -91,6 +91,6 @@
                 <samples>${lasers}</samples>
                 <resolution>1</resolution>
-                <min_angle>-${89.5*M_PI/180.0}</min_angle>
-                <max_angle>-${2.3125*M_PI/180.0}</max_angle>
+                <min_angle>${2.3125*M_PI/180.0}</min_angle>
+                <max_angle>${89.5*M_PI/180.0}</max_angle>
               </vertical>
             </scan>

Commit message: minor changes for flipper_auto mode

File: gazebo_description/models/NuBot_Pumbaa_v2/model_v2.urdf.xacro (robot description, xacro)
@@ -5,5 +5,5 @@
   <xacro:property name="track_mass" value="10" />
   <xacro:property name="flipper_mass" value="2.5" />
-  <xacro:property name="track_radius" value="0.09" />
+  <xacro:property name="track_radius" value="0.091" />
   <xacro:property name="track_width" value="0.18" />
   <xacro:property name="track_length" value="0.552" />
@@ -399,7 +399,7 @@
       <track_mu2>0.5</track_mu2>
       <!--The PID parameter of flippers position controll & initial position 1.5708 -->
-      <flip_p>1500</flip_p>
+      <flip_p>2000</flip_p>
       <flip_i>500</flip_i>
-      <flip_d>0</flip_d>
+      <flip_d>10</flip_d>
       <flip_initial>1.0472</flip_initial>
       <!--The parameters of tracks-->
