Commit message: add maintainer information

File: gazebo_description/models/NuBot_Pumbaa_v2/model_v2.urdf (robot description, URDF)
Before this commit: robot NuBot_Pumbaa_v2_rviz, 6 links, 5 joints
Links:
- added link imu_link, mass 0; collision box size=0.05 0.04 0.026; visual box size=0.05 0.04 0.026
- added link lidar_link, mass 0; collision cylinder length=0.11 radius=0.05; visual mesh filename=package://gazebo_description/models/RS_Bpearl/meshes/RS_Bpe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
Joints:
- added joint imu_joint: type fixed, parent base_link, child imu_link, origin xyz=-0.3185 0 0.133 rpy=0 0 3.1416, axis 0 0 0
- added joint lidar_joint: type fixed, parent base_link, child lidar_link, origin xyz=-0.36277 0 0.2115 rpy=0 1.508 3.1416, axis 0 0 0

Commit message: bug fix

File: gazebo_description/models/NuBot_Pumbaa_v2/model_v2.urdf (robot description, URDF)
Before this commit: robot NuBot_Pumbaa_v2_rviz, 8 links, 7 joints
Joints:
- joint lidar_joint: origin xyz=-0.36277 0 0.2115 rpy=0 1.508 3.1416 -> xyz=-0.36277 0 0.2115 rpy=0 1.5708 3.1416
