Commit message: fix twist direction bug

File: gazebo_description/models/IMU/model.urdf.xacro (robot description, xacro)
@@ -6,7 +6,7 @@
             <xacro:insert_block name="origin" />
             <parent link="${parent}"/>
-            <child link="${name}_link" />
+            <child link="${name}" />
         </joint>
-        <link name='${name}_link'>
+        <link name='${name}'>
             <!-- <inertial>
                 <mass value="0.1"/>
@@ -43,5 +43,5 @@
                 <robotNamespace>/</robotNamespace>
                 <updateRate>${hz}</updateRate>
-                <bodyName>${name}_link</bodyName>
+                <bodyName>${name}</bodyName>
                 <topicName>${topic}</topicName>
                 <accelDrift>0.005 0.005 0.005</accelDrift>

File: gazebo_description/models/RS_Bpearl/model_2.urdf.xacro (robot description, xacro)
@@ -6,7 +6,7 @@
       <xacro:insert_block name="origin" />
       <parent link="${parent}"/>
-      <child link="${name}_link"/>
+      <child link="${name}"/>
     </joint>
-    <link name='${name}_link'>
+    <link name='${name}'>
       <!-- <inertial>
         <origin xyz="0 -0.00079641 0.026317" rpy="0 0 0"/>
@@ -33,5 +33,5 @@
     </link>
     <!-- Gazebo requires the velodyne_gazebo_plugins package -->
-    <gazebo reference="${name}_link">
+    <gazebo reference="${name}">
       <xacro:if value="${gpu}">
         <sensor type="gpu_ray" name="${name}-RS_Bpearl">
@@ -67,5 +67,5 @@
           <plugin name="gazebo_ros_laser_controller" filename="libgazebo_ros_velodyne_gpu_laser.so">
             <topicName>${topic}</topicName>
-            <frameName>${name}_link</frameName>
+            <frameName>${name}</frameName>
             <organize_cloud>${organize_cloud}</organize_cloud>
             <min_range>${min_range}</min_range>
@@ -108,5 +108,5 @@
           <plugin name="gazebo_ros_laser_controller" filename="libgazebo_ros_velodyne_laser.so">
             <topicName>${topic}</topicName>
-            <frameName>${name}_link</frameName>
+            <frameName>${name}</frameName>
             <organize_cloud>${organize_cloud}</organize_cloud>
             <min_range>${min_range}</min_range>

File: gazebo_description/models/RS_Helios_5515/model_2.urdf.xacro (robot description, xacro)
@@ -6,7 +6,7 @@
       <xacro:insert_block name="origin" />
       <parent link="${parent}"/>
-      <child link="${name}_link"/>
+      <child link="${name}"/>
     </joint>
-    <link name="${name}_link">
+    <link name="${name}">
       <!-- <inertial>
         <origin xyz="0 0 0" rpy="0 0 0"/>
@@ -33,5 +33,5 @@
     </link>
     <!-- Gazebo requires the velodyne_gazebo_plugins package -->
-    <gazebo reference="${name}_link">
+    <gazebo reference="${name}">
       <xacro:if value="${gpu}">
         <sensor type="gpu_ray" name="${name}-RS_Helios_5515">
@@ -67,5 +67,5 @@
           <plugin name="gazebo_ros_laser_controller" filename="libgazebo_ros_velodyne_gpu_laser.so">
             <topicName>${topic}</topicName>
-            <frameName>${name}_link</frameName>
+            <frameName>${name}</frameName>
             <organize_cloud>${organize_cloud}</organize_cloud>
             <min_range>${min_range}</min_range>
@@ -108,5 +108,5 @@
           <plugin name="gazebo_ros_laser_controller" filename="libgazebo_ros_velodyne_laser.so">
             <topicName>${topic}</topicName>
-            <frameName>${name}_link</frameName>
+            <frameName>${name}</frameName>
             <organize_cloud>${organize_cloud}</organize_cloud>
             <min_range>${min_range}</min_range>

Commit message: fix bugs

File: gazebo_description/models/IMU/model.urdf.xacro (robot description, xacro)
@@ -24,19 +24,32 @@
             </geometry>
             </collision>
-            <!-- <sensor name='imu_sensor' type='imu'>
+        </link>
+        <!-- <gazebo reference="${name}">
+            <gravity>true</gravity>
+            <sensor name='imu_sensor' type='imu'>
                 <always_on>true</always_on>
-                <update_rate>50</update_rate>
+                <update_rate>${hz}</update_rate>
                 <visualize>true</visualize>
+                <pose>0 0 0 0 0 0</pose>
                 <plugin filename='libgazebo_ros_imu_sensor.so' name='imu_plugin'>
-                    <topicName>imu</topicName>
-                    <updateRateHZ>100.0</updateRateHZ>
+                    <topicName>${topic}</topicName>
+                    <updateRateHZ>${hz}</updateRateHZ>
                     <gaussianNoise>0.0</gaussianNoise>
                     <xyzOffset>0 0 0</xyzOffset>
                     <rpyOffset>0 0 0</rpyOffset>
-                    <frameName>imu</frameName>
+                    <frameName>${name}</frameName>
                 </plugin>
-                <pose>0 0 0 0 0 0</pose>
-            </sensor> -->
-        </link>
+            </sensor>
+        </gazebo> -->
+        <!-- <gazebo>
+            <plugin name="imu_plugin" filename="libgazebo_ros_imu.so">
+                <alwaysOn>true</alwaysOn>
+                <bodyName>${name}</bodyName>
+                <topicName>${topic}</topicName>
+                <serviceName>${topic}_service</serviceName>
+                <gaussianNoise>0.0</gaussianNoise>
+                <updateRate>400.0</updateRate>
+            </plugin>
+        </gazebo> -->
         <gazebo>
             <plugin name="imu_controller" filename="libhector_gazebo_ros_imu.so">

File: gazebo_description/models/NuBot_Pumbaa_v2/model_v2.urdf.xacro (robot description, xacro)
@@ -64,7 +64,9 @@
     <mu1>1</mu1>
     <mu2>1</mu2>
-    <fdir1 value="0 1 0" />
-    <gravity>1</gravity>
-    <maxContacts>10</maxContacts>
+    <kp value="10000000.0" />
+    <kd value="1.0" />
+    <fdir1 value="0 1 0" />
+    <gravity>1</gravity>
+    <maxContacts>2</maxContacts>
   </gazebo>
   <!--left_track-->
@@ -106,7 +108,9 @@
     <mu1>0.7</mu1>
     <mu2>150</mu2>
-    <fdir1 value="0 1 0" />
-    <gravity>1</gravity>
-    <maxContacts>10</maxContacts>
+    <kp value="10000000.0" />
+    <kd value="1.0" />
+    <fdir1 value="0 1 0" />
+    <gravity>1</gravity>
+    <maxContacts>2</maxContacts>
   </gazebo>
   <!--left_track joints-->
@@ -157,7 +161,9 @@
     <mu1>0.7</mu1>
     <mu2>150</mu2>
-    <fdir1 value="0 1 0" />
-    <gravity>1</gravity>
-    <maxContacts>10</maxContacts>
+    <kp value="10000000.0" />
+    <kd value="1.0" />
+    <fdir1 value="0 1 0" />
+    <gravity>1</gravity>
+    <maxContacts>2</maxContacts>
   </gazebo>
   <!--right_track joints-->
@@ -208,7 +214,9 @@
     <mu1>0.7</mu1>
     <mu2>150</mu2>
-    <fdir1 value="0 1 0" />
-    <gravity>1</gravity>
-    <maxContacts>10</maxContacts>
+    <kp value="10000000.0" />
+    <kd value="1.0" />
+    <fdir1 value="0 1 0" />
+    <gravity>1</gravity>
+    <maxContacts>2</maxContacts>
   </gazebo>
   <joint name='rear_left_flipper_joint' type='revolute'>
@@ -257,7 +265,9 @@
     <mu1>0.7</mu1>
     <mu2>150</mu2>
-    <fdir1 value="0 1 0" />
-    <gravity>1</gravity>
-    <maxContacts>10</maxContacts>
+    <kp value="10000000.0" />
+    <kd value="1.0" />
+    <fdir1 value="0 1 0" />
+    <gravity>1</gravity>
+    <maxContacts>2</maxContacts>
   </gazebo>
   <joint name='rear_right_flipper_joint' type='revolute'>
@@ -306,7 +316,9 @@
     <mu1>0.7</mu1>
     <mu2>150</mu2>
-    <fdir1 value="0 1 0" />
-    <gravity>1</gravity>
-    <maxContacts>10</maxContacts>
+    <kp value="10000000.0" />
+    <kd value="1.0" />
+    <fdir1 value="0 1 0" />
+    <gravity>1</gravity>
+    <maxContacts>2</maxContacts>
   </gazebo>
   <joint name='front_left_flipper_joint' type='revolute'>
@@ -355,7 +367,9 @@
     <mu1>0.7</mu1>
     <mu2>150</mu2>
-    <fdir1 value="0 1 0" />
-    <gravity>1</gravity>
-    <maxContacts>10</maxContacts>
+    <kp value="10000000.0" />
+    <kd value="1.0" />
+    <fdir1 value="0 1 0" />
+    <gravity>1</gravity>
+    <maxContacts>2</maxContacts>
   </gazebo>
   <joint name='front_right_flipper_joint' type='revolute'>
@@ -388,5 +402,5 @@
       <flip_i>100</flip_i>
       <flip_d>0</flip_d>
-      <flip_initial>1.5708</flip_initial>
+      <flip_initial>1.0472</flip_initial>
       <!--The parameters of tracks-->
       <tracksSeparation>0.29</tracksSeparation>
@@ -397,22 +411,22 @@
   </gazebo>
   <!-- RS-Helios includes -->
-  <xacro:include filename="$(find gazebo_description)/models/RS_Helios_5515/model_2.urdf.xacro"/>
+  <!-- <xacro:include filename="$(find gazebo_description)/models/RS_Helios_5515/model_2.urdf.xacro"/>
   <xacro:RS_Helios_5515 parent="chassis_link" name="rs_helios" topic="/lidar_points" hz="10" samples="1800" min_angle="-${PI}" max_angle="${PI}" min_range ="0.2" max_range="50.0" gpu="true">
     <origin xyz="-0.221 0 0.2545" rpy="0 0 ${PI}" />
-  </xacro:RS_Helios_5515>
+  </xacro:RS_Helios_5515> -->
   <!-- IMU includes (RS-Helios) -->
+  <!-- <xacro:include filename="$(find gazebo_description)/models/IMU/model.urdf.xacro"/>
+  <xacro:IMU parent="chassis_link" name="imu" topic="/imu/data" hz="400">
+    <origin xyz="-0.221 0 0.131" rpy="0 0 ${PI}" />
+  </xacro:IMU> -->
+  <!-- RS-Bpearl includes -->
+  <xacro:include filename="$(find gazebo_description)/models/RS_Bpearl/model_2.urdf.xacro"/>
+  <xacro:RS_Bpearl parent="chassis_link" name="rs_bpearl" topic="/velodyne_points" hz="10" lasers="32" samples="1800" min_angle="-${PI}" max_angle="${PI}" min_range ="0.1" max_range="50.0" gpu="true"> <!-- lidar_points -->
+    <origin xyz="-0.36277 0 0.2115" rpy="0 ${PI/2} ${PI}" />
+  </xacro:RS_Bpearl>
+  <!-- IMU includes (RS-Bpearl) -->
   <xacro:include filename="$(find gazebo_description)/models/IMU/model.urdf.xacro"/>
   <xacro:IMU parent="chassis_link" name="imu" topic="/imu/data" hz="400">
-    <origin xyz="-0.221 0 0.131" rpy="0 0 ${PI}" />
+    <origin xyz="-0.3185 0 0.133" rpy="0 0 ${PI}" />
   </xacro:IMU>
-  <!-- RS-Bpearl includes -->
-  <!-- <xacro:include filename="$(find gazebo_description)/models/RS_Bpearl/model_2.urdf.xacro"/>
-  <xacro:RS_Bpearl parent="chassis_link" name="rs_bpearl" topic="/lidar_points" hz="10" lasers="32" samples="1800" min_angle="-${PI}" max_angle="${PI}" min_range ="0.1" max_range="50.0" gpu="true">
-    <origin xyz="-0.36277 0 0.2115" rpy="${PI} ${PI/2} 0" />
-  </xacro:RS_Bpearl> -->
-  <!-- IMU includes (RS-Bpearl) -->
-  <!-- <xacro:include filename="$(find gazebo_description)/models/IMU/model.urdf.xacro"/>
-  <xacro:IMU parent="chassis_link" name="imu" topic="/imu/data" hz="400">
-    <origin xyz="-0.3185 0 0.133" rpy="0 0 ${PI}" />
-  </xacro:IMU> -->
 </robot>

File: gazebo_description/models/RS_Bpearl/model_2.urdf.xacro (robot description, xacro)
@@ -26,5 +26,5 @@
       </collision>
       <visual name='visual'>
-        <origin xyz="0 0 0" rpy="${M_PI} 0 0"/>
+        <origin xyz="0 0 0" rpy="0 0 0"/>
         <geometry>
           <mesh filename="model://RS_Bpearl/meshes/RS_Bpearl_frame.STL" />

Commit message: add stairs & refine parameteres

File: gazebo_description/models/IMU/model.urdf.xacro (robot description, xacro)
@@ -1,16 +1,16 @@
-<?xml version="1.0" ?>
+<?xml version="1.0"?>
 <robot xmlns:xacro="http://www.ros.org/wiki/xacro" name="IMU">
     <xacro:property name="M_PI" value="3.1415926535897931" />
     <xacro:macro name="IMU" params="*origin parent:=base_link name:=imu topic:=/imu/data hz:=400">
-        <joint name="${name}_mount_joint" type='fixed'>
+        <joint name="${name}_mount_joint" type="fixed">
             <xacro:insert_block name="origin" />
             <parent link="${parent}"/>
             <child link="${name}" />
         </joint>
-        <link name='${name}'>
+        <link name="${name}">
             <!-- <inertial>
                 <mass value="0.1"/>
             </inertial> -->
-            <visual name='visual'>
+            <visual name="visual">
                 <origin xyz="0 0 0.013" rpy="0 0 0"/>
                 <geometry>
@@ -18,5 +18,5 @@
                 </geometry>
             </visual>
-            <collision name='collision'>
+            <collision name="collision">
             <origin xyz="0 0 0.013" rpy="0 0 0"/>
             <geometry>
@@ -35,5 +35,5 @@
                     <topicName>${topic}</topicName>
                     <updateRateHZ>${hz}</updateRateHZ>
-                    <gaussianNoise>0.0</gaussianNoise>
+                    <gaussianNoise>0.005</gaussianNoise>
                     <xyzOffset>0 0 0</xyzOffset>
                     <rpyOffset>0 0 0</rpyOffset>
@@ -48,6 +48,6 @@
                 <topicName>${topic}</topicName>
                 <serviceName>${topic}_service</serviceName>
-                <gaussianNoise>0.0</gaussianNoise>
-                <updateRate>400.0</updateRate>
+                <gaussianNoise>0.005</gaussianNoise>
+                <updateRate>${hz}</updateRate>
             </plugin>
         </gazebo> -->

File: gazebo_description/models/NuBot_Pumbaa_v2/model_v2.urdf.xacro (robot description, xacro)
@@ -399,6 +399,6 @@
       <track_mu2>0.8</track_mu2>
       <!--The PID parameter of flippers position controll & initial position 1.5708 -->
-      <flip_p>1500</flip_p>
-      <flip_i>100</flip_i>
+      <flip_p>1750</flip_p>
+      <flip_i>800</flip_i>
       <flip_d>0</flip_d>
       <flip_initial>0</flip_initial><!--1.0472-->

File: gazebo_description/models/RS_Bpearl/model_2.urdf.xacro (robot description, xacro)
@@ -62,5 +62,5 @@
               <type>gaussian</type>
               <mean>0.0</mean>
-              <stddev>0.0</stddev>
+              <stddev>${noise}</stddev>
             </noise>
           </ray>
@@ -103,5 +103,5 @@
               <type>gaussian</type>
               <mean>0.0</mean>
-              <stddev>0.0</stddev>
+              <stddev>${noise}</stddev>
             </noise>
           </ray>

File: gazebo_description/models/RS_Helios_5515/model_2.urdf.xacro (robot description, xacro)
@@ -62,5 +62,5 @@
               <type>gaussian</type>
               <mean>0.0</mean>
-              <stddev>0.0</stddev>
+              <stddev>${noise}</stddev>
             </noise>
           </ray>
@@ -103,5 +103,5 @@
               <type>gaussian</type>
               <mean>0.0</mean>
-              <stddev>0.0</stddev>
+              <stddev>${noise}</stddev>
             </noise>
           </ray>
